Commit message: MOD: In robot model add two front wheels, deactivate small castor wheel 	changed:       ros_101_gazebo_rviz/urdf/robot_tutorial.xacro
MOD: Add new wheels in differential drive gazebo plugin
	changed:       ros_101_gazebo_rviz/urdf/robot_tutorial_gazebo.xacro

File: ros_101_gazebo_rviz/urdf/robot_tutorial.xacro (robot description, xacro)
@@ -2,9 +2,9 @@
 <robot xmlns:xacro="http://www.ros.org/wiki/xacro" name="robot_tutorial">
   <xacro:property name="base_width" value="0.16"/>
-  <xacro:property name="base_len" value="0.16"/>
+  <xacro:property name="base_len" value="0.26"/>
   <xacro:property name="wheel_radius" value="0.035"/>
   <xacro:property name="base_wheel_gap" value="0.007"/>
   <xacro:property name="wheel_separation" value="0.15"/>
-  <xacro:property name="wheel_joint_offset" value="0.02"/>
+  <xacro:property name="wheel_joint_offset" value="0.07"/>
   <xacro:property name="caster_wheel_radius" value="${wheel_radius/2}"/>
   <xacro:property name="caster_wheel_mass" value="0.001"/>
@@ -74,5 +74,5 @@
   </joint>
   <!--Wheel link & joint macro-->
-  <xacro:macro name="wheel" params="prefix reflect">
+  <xacro:macro name="wheel" params="prefix reflect_x reflect_y">
     <link name="${prefix}_wheel">
       <visual>
@@ -95,11 +95,14 @@
       <parent link="base_link"/>
       <child link="${prefix}_wheel"/>
-      <origin xyz="${wheel_joint_offset} ${((base_width/2)+base_wheel_gap)*reflect} -0.005" rpy="0 0 0"/>
+      <origin xyz="${wheel_joint_offset*reflect_x} ${((base_width/2)+base_wheel_gap)*reflect_y} -0.005" rpy="0 0 0"/>
     </joint>
   </xacro:macro>
   <!--Create Left & Right Wheel links/joints-->
-  <xacro:wheel prefix="left" reflect="1"/>
-  <xacro:wheel prefix="right" reflect="-1"/>
+  <xacro:wheel prefix="left_front" reflect_x="1" reflect_y="1"/>
+  <xacro:wheel prefix="right_front" reflect_x="1" reflect_y="-1"/>
+  <xacro:wheel prefix="left_back" reflect_x="-1" reflect_y="1"/>
+  <xacro:wheel prefix="right_back" reflect_x="-1" reflect_y="-1"/>
   <!--Caster Wheel Link-->
+  <!--
   <link name="caster_wheel">
     <visual>
@@ -118,5 +121,7 @@
     <xacro:sphere_inertia m="10" r="${caster_wheel_radius}"/>
   </link>
+   -->
   <!--Caster Wheel Joint-->
+  <!--
   <joint name="caster_wheel_joint" type="continuous">
     <axis xyz="0 1 0" rpy="0 0 0" />
@@ -125,4 +130,5 @@
     <origin xyz="${caster_wheel_joint_offset} 0 -${caster_wheel_radius+0.005}" rpy="0 0 0"/>
   </joint>
+   -->
   <xacro:include filename="$(find ros_101_gazebo_rviz)/urdf/robot_tutorial_gazebo.xacro"/>
 </robot>

File: ros_101_gazebo_rviz/urdf/robot_tutorial_gazebo.xacro (robot description, xacro)
@@ -6,6 +6,8 @@
       <legacyMode>false</legacyMode>
       <updateRate>20</updateRate>
-      <leftJoint>left_wheel_joint</leftJoint>
-      <rightJoint>right_wheel_joint</rightJoint>
+      <leftJoint>left_front_wheel_joint</leftJoint>
+      <leftJoint>left_back_wheel_joint</leftJoint>
+      <rightJoint>right_front_wheel_joint</rightJoint>
+      <rightJoint>right_back_wheel_joint</rightJoint>
       <wheelSeparation>${wheel_separation}</wheelSeparation>
       <wheelDiameter>${wheel_radius * 2}</wheelDiameter>
